File: eagle/BaseMachine_Sequencer_UI/BaseMachine_Sequencer_UI.brd (EAGLE design)
At the start: 93.7 x 71.1 mm, 12 parts, among them SW1 ALPS_SKHCBFA010, SW5 AK_TCTSW, SW6 AK_TCTSW

Commit message: Update parts position
Parts:
- added LED1: (no value), led:LED3MM
- added R1: (no value), rcl:0207/7
- JP1: device pinhead:1X07/90 -> pinhead:1X06/90
- JP2: device pinhead:1X05/90 -> pinhead:1X08/90
- moved JP1 5.68 mm to (15.2, 69.8)
- moved JP2 3.59 mm to (63.5, 69.8)
- moved JP3 2.54 mm to (41.9, 69.8)
- moved LCD1 2.54 mm to (20.3, 19.1)
- moved U$3 1.80 mm to (85.1, 17.8), turned to 180 degrees
- turned SW5 to 0 degrees
- turned SW6 to 0 degrees
Connections:
- removed net N$11: JP2.5, RE2.P$4
- removed net N$18: JP3.3, LCD1.3
- removed net N$5: JP2.3, RE1.P$4
- new net N$10: JP1.1, RE1.P$2
- new net N$13: JP1.2, RE1.P$4
- new net N$9: LED1.A, R1.2
- new net VDD: JP3.3, LCD1.3, R1.1
- net GND: now also LED1.K; no longer JP1.7, JP2.1
- net N$12: now also JP1.3; no longer JP1.1
- net N$19: now also JP1.4; no longer JP1.2
- net N$2: now also JP2.3; no longer JP1.5
- net N$3: now also JP2.6, RE2.P$4; no longer JP2.2, RE1.P$2
- net N$4: now also JP2.1; no longer JP1.3
- net N$6: now also JP2.2; no longer JP1.4
- net N$7: now also JP2.5; no longer JP2.4
- net N$8: now also JP2.4; no longer JP1.6

Commit message: routing
Parts:
- R1: value (none) -> 1k
Changed lines of the file:
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@@
 <element name="U$2" library="mylib2" package="ALPS_SKHCBFA010" value="ALPS_SKHCBFA010" x="67.31" y="7.62" rot="R180"/>
 <element name="U$3" library="mylib2" package="ALPS_SKHCBFA010" value="ALPS_SKHCBFA010" x="85.09" y="17.78" rot="R180"/>
-<element name="R1" library="rcl" package="0207/7" value="" x="80.01" y="68.58"/>
+<element name="R1" library="rcl" package="0207/7" value="1k" x="80.01" y="68.58"/>
 <element name="LED1" library="led" package="LED3MM" value="" x="86.36" y="67.31" rot="R270"/>
 <element name="JP1" library="pinhead" package="1X06/90" value="" x="15.24" y="69.85"/>

Commit message: Update: UI & UI2 Board Design
Parts:
- removed LCD1: ATD_CH12864F-SPI, mylib2:ATD-CH12864F-SPI
- removed LED1: (no value), led:LED3MM
- removed R1: 1k, rcl:0207/7
- added U$4: ATD_CH12864F-SPI, mylib2:ATD-CH12864F-SPI
- JP1: value (none) -> SW1
- JP2: value (none) -> SW2; device pinhead:1X08/90 -> pinhead:1X07/90
- moved JP2 2.54 mm to (61.0, 69.8)
- moved SW5 2.54 mm to (7.62, 29.2)
- moved SW6 2.54 mm to (7.62, 16.5)
- moved JP1 1.27 mm to (14.0, 69.8)
- moved RE2 1.27 mm to (86.4, 50.8), turned to 180 degrees
- turned RE1 to 180 degrees
Connections:
- removed net N$1: JP3.1, LCD1.1
- removed net N$20: JP3.5, LCD1.5
- removed net N$21: JP3.6, LCD1.6
- removed net N$7 (its old number): JP2.5, RE2.P$2
- new net LCD1: JP3.1, U$4.1
- new net N$3: JP2.7, RE2.P$2
- new net N$5: JP3.3, U$4.3
- net GND: now also JP1.5, JP2.1, JP3.5, U$4.5; no longer JP3.4, LCD1.4, LED1.K
- net N$10: now also RE1.P$4; no longer RE1.P$2
- net N$13: now also RE1.P$2; no longer RE1.P$4
- net N$17: now also U$4.2; no longer LCD1.2
- net N$2: now also JP2.4; no longer JP2.3
- net N$22: now also U$4.7; no longer LCD1.7
- net N$23: now also U$4.8; no longer LCD1.8
- net N$4: now also JP2.2; no longer JP2.1
- net N$6: now also JP2.3; no longer JP2.2
- net N$8: now also JP2.5; no longer JP2.4
- net N$9: now also JP3.4, U$4.4; no longer LED1.A, R1.2
- net VDD: now also JP1.6, JP3.6, U$4.6; no longer JP3.3, LCD1.3, R1.1
Routing:
- net GND: track 0.00 -> 315.3 mm
- net N$4: track 0.00 -> 85.9 mm
- net VDD: track 0.00 -> 78.7 mm
- net N$6: track 0.00 -> 69.6 mm
- net N$2: track 0.00 -> 68.6 mm
- net N$8: track 0.00 -> 64.7 mm
- net N$19: track 0.00 -> 57.5 mm
- net N$9: track 0.00 -> 48.3 mm
- net N$5: track 0.00 -> 48.3 mm
- net N$23: track 0.00 -> 48.3 mm
- net N$22: track 0.00 -> 48.3 mm
- net N$17: track 0.00 -> 48.3 mm
- net LCD1: track 0.00 -> 48.3 mm
- net N$12: track 0.00 -> 43.8 mm
- net N$3: track 0.00 -> 23.9 mm
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Other:
- board text added: "VDDのジャンパは未実装"
